File: schematics/65816/65816.kicad_sch (KiCad schematic)
At the start: 2 parts

Commit message: schematics
Parts:
- added X1: CXO_DIP8, Oscillator:Oscillator_DIP-8, symbol Oscillator:CXO_DIP8
- U2: renamed from U?; value W65C22NxP -> (none)
- gave numbers to parts that had none: 1
Connections:
- net +5V: now also X1.8 (Vcc)
- net D0: now also U2.33 (D0)
- net D1: now also U2.32 (D1)
- net GND: now also X1.4 (GND)
- net D7: now reaches U2.26 (D7)
- net D7: now also U1.26 (D7)
- net D6: now reaches U2.27 (D6)
- net D6: now also U1.27 (D6)
- net D5: now reaches U2.28 (D5)
- net D5: now also U1.28 (D5)
- net D4: now reaches U2.29 (D4)
- net D4: now also U1.29 (D4)
- net D3: now reaches U2.30 (D3)
- net D3: now also U1.30 (D3)
- net D2: now reaches U2.31 (D2)
- net D2: now also U1.31 (D2)
- net A1: now reaches U1.10 (A1)
- net A2: now reaches U1.11 (A2)
- net A3: now reaches U1.12 (A3)
- net A4: now reaches U1.13 (A4)
- net A5: now reaches U1.14 (A5)
- net A6: now reaches U1.15 (A6)
- net A7: now reaches U1.16 (A7)
- net A8: now reaches U1.17 (A8)
- net A9: now reaches U1.18 (A9)
- net A10: now reaches U1.19 (A10)
- net A10: no longer U1.20 (A11)
- net A12: now reaches U1.22 (A12)
- net A13: now reaches U1.23 (A13)
- net A14: now reaches U1.24 (A14)
- net A15: now reaches U1.25 (A15)
- net CLK: now reaches U1.37 (ϕ0)
- net ~{RES}: now reaches U1.40 (~{RES})
- net A0: now reaches U1.9 (A0)
- new net A11: U1.20 (A11)
- no-connect marks 0 -> 1
Other:
- company: (none) -> Alexander Hansen
- title: (none) -> 65816
- moved on the sheet: U2

Commit message: schematics
Parts:
- added R?: 3.9K, symbol Device:R
- U2: value (none) -> 65C22
Connections:
- net +5V: now also X1.1 (EN), R?.1
- net A0: now also U2.38 (RS0)
- net A1: now also U2.37 (RS1)
- net A2: now also U2.36 (RS2)
- net A3: now also U2.35 (RS3)
- net KBD0: now reaches U2.2 (PA0)
- net KBD1: now reaches U2.3 (PA1)
- net KBD2: now reaches U2.4 (PA2)
- net KB_INT: now reaches U2.40 (CA1)
- net KBD3: now reaches U2.5 (PA3)
- net KBD4: now reaches U2.6 (PA4)
- net KBD5: now reaches U2.7 (PA5)
- net KBD6: now reaches U2.8 (PA6)
- net KBD7: now reaches U2.9 (PA7)
- net at U1.2 (RDY): now also R?.2
- net ~{IRQ}: now reaches U1.4 (~{IRQ})
Other:
- added sheet Keyboard (ps2.kicad_sch)

Commit message: schematics
Parts:
- added C?: (no value), symbol Device:C
- added D?: (no value), symbol Diode:1N4148
- added J?: (no value), symbol Connector:Mini-DIN-6
- added R?: (no value), symbol Device:R_US
- added U? (x2): (no value), symbol 74xx:74HC595
- added U? (x3): (no value), symbol 74xx:74HC14
- added U?: ATF22V10C-15PU, 24P3_ATM, symbol 2022-03-21_20-19-29:ATF22V10C-15PU
- X1: value CXO_DIP8 -> (none)
Connections:
- net +5V: now also J?.4, U?.10 (~{SRCLR}), U?.10 (~{SRCLR}), U?.16 (VCC), U?.16 (VCC), U?.24 (VCC)
- net A10: now also U?.9 (IN)
- net A11: now also U?.8 (IN)
- net A12: now also U?.7 (IN)
- net A13: now also U?.6 (IN)
- net A14: now also U?.5 (IN)
- net A15: now also U?.4 (IN/PD)
- net A8: now also U?.11 (IN)
- net A9: now also U?.10 (IN)
- net GND: now also C?.2, J?.3, U?.12 (GND), U?.13 (~{OE}), U?.13 (~{OE}), U?.8 (GND), U?.8 (GND)
- net KB_INT: now also U?.12 (RCLK), U?.12 (RCLK), U?.4
- net ~{IRQ}: now also U2.21 (~{IRQ})
- net R/~{W}: now reaches U2.22 (R/~{W})
- net R/~{W}: now also U1.34 (R/~{W})
- net KBD0 renamed KB_D0
- net KB_D0: now also U?.1 (QB)
- net KBD1 renamed KB_D1
- net KB_D1: now also U?.15 (QA)
- net KBD2 renamed KB_D2
- net KB_D2: now also U?.7 (QH)
- net KBD3 renamed KB_D3
- net KB_D3: now also U?.6 (QG)
- net KBD4 renamed KB_D4
- net KB_D4: now also U?.5 (QF)
- net KBD5 renamed KB_D5
- net KB_D5: now also U?.4 (QE)
- net KBD6 renamed KB_D6
- net KB_D6: now also U?.3 (QD)
- net KBD7 renamed KB_D7
- net KB_D7: now also U?.2 (QC)
- new net: U?.11 (SRCLK), U?.11 (SRCLK), U?.2
- new net: U?.14 (SER), U?.9 (QH')
- new net: D?.2 (A), R?.1, U?.4
- new net: C?.1, D?.1 (K), R?.2, U?.3
- new net A16: U?.3 (IN)
- new net A17: U?.2 (IN)
- new net A18: U?.1 (CLK/IN)
- new net IO1_CS: U?.19 (I/O)
- new net IO2_CS: U?.20 (I/O)
- new net IO3_CS: U?.21 (I/O)
- new net IO4_CS: U?.22 (I/O)
- new net KB_CLK: J?.5, U?.1, U?.3
- new net KB_DATA: J?.1, U?.14 (SER)
- new net RAM_CS: U?.23 (I/O)
- new net ROM_CS: U?.18 (I/O)
- no-connect marks 1 -> 17
Other:
- removed sheet Keyboard
- moved on the sheet: R?, U1, U2, X1

Commit message: kicad work
Parts:
- added U3: AS6C4008-55PCN, Alliance_Memory-AS6C4008-55PCN-0-0-*, symbol eec:AS6C4008-55PCN
- added U4: 74HC573, symbol 74xx:74LS573
- C?: value (none) -> 0.01 uF
- D?: value (none) -> 1N4148; footprint (none) -> Diode_THT:D_DO-35_SOD27_P7.62mm_Horizontal
- J?: value (none) -> Keyboard
- R?: value (none) -> 33K
- U? (x2): value (none) -> 74HC595
- U? (x3): value (none) -> 74HC14
- X1: value (none) -> 10.000MHz
- gave numbers to parts that had none: 1
Connections:
- net IO1_CS is gone; now on net ~{IO1_CS}: U0.19 (I/O)
- net +5V: now also U2.24 (CS1), U3.32 (Vcc), U4.20 (VCC)
- net A0: now also U3.12 (A0)
- net A1: now also U3.11 (A1)
- net A10: now also U3.23 (A10)
- net A11: now also U3.25 (A11)
- net A12: now also U3.4 (A12)
- net A13: now also U3.28 (A13)
- net A14: now also U3.3 (A14)
- net A15: now also U3.31 (A15)
- net A16: now also U3.2 (A16), U4.19 (Q0)
- net A17: now also U3.30 (A17), U4.18 (Q1)
- net A18: now also U3.1 (A18), U4.17 (Q2)
- net A2: now also U3.10 (A2)
- net A3: now also U3.9 (A3)
- net A4: now also U3.8 (A4)
- net A5: now also U3.7 (A5)
- net A6: now also U3.6 (A6)
- net A7: now also U3.5 (A7)
- net A8: now also U3.27 (A8)
- net A9: now also U3.26 (A9)
- net D0: now also U3.13 (DQ0), U4.2 (D0)
- net D1: now also U3.14 (DQ1), U4.3 (D1)
- net D2: now also U3.15 (DQ2), U4.4 (D2)
- net D3: now also U3.17 (DQ3), U4.5 (D3)
- net D4: now also U3.18 (DQ4), U4.6 (D4)
- net D5: now also U3.19 (DQ5), U4.7 (D5)
- net D6: now also U3.20 (DQ6), U4.8 (D6)
- net D7: now also U3.21 (DQ7), U4.9 (D7)
- net GND: now also U3.16 (Vss), U4.1 (OE), U4.10 (GND)
- net RAM_CS: now also U3.22 (~{CE}); no longer U0.23 (I/O)
- net R/~{W}: now also U3.29 (~{WE})
- net ~{IO1_CS}: now reaches U2.23 (~{CS2})
- net IO2_CS renamed ~{IO2_CS}
- net IO3_CS renamed ~{IO3_CS}
- net IO4_CS renamed ~{IO4_CS}
- net ROM_CS renamed ~{ROM_CS}
- new net A19: U4.16 (Q3)
- new net A20: U4.15 (Q4)
- new net A21: U4.14 (Q5)
- new net A22: U4.13 (Q6)
- new net A23: U4.12 (Q7)
- new net DB_LOAD: U4.11 (Load)
- new net ~{RAM_CS}: U0.23 (I/O)
Other:
- moved on the sheet: U2

Commit message: schematics
Connections:
- net CLK: now also U2.25 (ϕ2)
- net ~{RES}: now also U2.34 (~{RES})
Changed lines of the file:
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@@
+    (stroke (width 0) (type default) (color 0 0 0 0))
+  )
+  (wire (pts (xy 176.53 134.62) (xy 180.34 134.62))
     (stroke (width 0) (type default) (color 0 0 0 0))
   )
@@
     (stroke (width 0) (type default) (color 0 0 0 0))
   )
-  (wire (pts (xy 175.26 142.24) (xy 180.34 142.24))
+  (wire (pts (xy 176.53 142.24) (xy 180.34 142.24))
     (stroke (width 0) (type default) (color 0 0 0 0))
   )
@@
   )
   (wire (pts (xy 142.24 80.01) (xy 149.86 80.01))
+    (stroke (width 0) (type default) (color 0 0 0 0))
+  )
+  (wire (pts (xy 176.53 137.16) (xy 180.34 137.16))
     (stroke (width 0) (type default) (color 0 0 0 0))
   )
@@
     )
   )
-  (global_label "~{IRQ}" (shape input) (at 175.26 142.24 180) (fields_autoplaced)
+  (global_label "~{IRQ}" (shape input) (at 176.53 142.24 180) (fields_autoplaced)
     (effects (font (size 1.27 1.27)) (justify right))
-    (property "Intersheet References" "${INTERSHEET_REFS}" (id 0) (at 169.6417 142.1606 0)
+    (property "Intersheet References" "${INTERSHEET_REFS}" (id 0) (at 170.9117 142.1606 0)
+      (effects (font (size 1.27 1.27)) (justify right) hide)
+    )
+  )
+  (global_label "CLK" (shape input) (at 176.53 137.16 180) (fields_autoplaced)
+    (effects (font (size 1.27 1.27)) (justify right))
+    (property "Intersheet References" "${INTERSHEET_REFS}" (id 0) (at 170.5488 137.0806 0)
       (effects (font (size 1.27 1.27)) (justify right) hide)
     )
@@
       (effects (font (size 1.27 1.27)) (justify right) hide)
     )
+  )
+  (global_label "~{RES}" (shape input) (at 176.53 134.62 180) (fields_autoplaced)
+    (effects (font (size 1.27 1.27)) (justify right))
+    (property "Intersheet References" "${INTERSHEET_REFS}" (id 0) (at 170.4883 134.5406 0)
+      (effects (font (size 1.27 1.27)) (justify right) hide)
+    )
